File: PDB.sch (EAGLE design)
At the start: 65 parts, among them J1 B06B-HCMKK, J2 B06B-HCMKK, J3 SS-6488-NF-A431, J4 SS-6488-NF-A431, J5 B06B-HCMKK, J6 B03B-HCMKS, J7 B03B-HCMKS

Commit message: Schemetic first draft done
Parts:
- removed 555_CLK_LED, _ADD1, _ADD2, _EXT_CLK: (no value), led:LEDCHIPLED_0805
- removed ADD1: NCV8405ADPAK-3PIN, master_library:NCV8405ADPAK-3PIN
- removed ADD1_: (no value), switch:M9040P
- removed JP2: (no value), jumper:JP2E
- removed LIGHTS: 8-PIN-MOLEX-RA-FEMALE, master_library:8-PIN-MOLEX-RA-FEMALE
- removed R13: 220, rcl:R-US_R0805
- removed R17: 470, resistor:R-US_R3225
- removed R2: 4.7K, rcl:R-US_R0805
- removed R23: 100, resistor:R-US_R0805
- removed R24, R25: 710, master_library:R-US_R0805
- removed TP3: PTR1B2,54, testpad:PTR1B2,54
- removed U$1: JST-PH_5-PIN_HEADER, master_library:JST-PH_5-PIN_HEADER
- added J8: SS-6488-NF-A431, AUX Lib:SS-6488-NF-A431
Connections:
- removed net 555_OUT: 555_CLK_LED.A, JP2.1
- removed net EXT_CLK: JP2.3, U$1.2, _EXT_CLK.A
- removed net H5: ADD1_.P, R13.1
- removed net N$2: 555_CLK_LED.C, R17.1
- removed net N$26: ADD1.G, R13.2, R2.1, TP3.TP
- removed net N$3: R23.1, _EXT_CLK.C
- removed net N$4: R24.1, _ADD1.C
- removed net N$5: R25.1, _ADD2.C
- removed net µC_ADD_1: ADD1_.O, U$1.4, _ADD1.A
- removed net µC_ADD_2: U$1.3, _ADD2.A
- new net CLK_SW: J8.4, U$3.D2/PWM
- new net CS: J8.6, U$3.D4/SDA2/CAN0RX/PWM
- new net DC: J8.5, U$3.D5/(MISO)/(TX1)/PWM
- new net MOSI_SW: J8.3, U$3.D3/SCL2/CAN0TX/PWM
- new net RESET: J8.7, U$3.D6/PWM
- net 10V_REG: no longer ADD1_.S
- net 3.3V: now also U$3.3V3@1
- net 5V_REG: now also J8.1
- net BRAKE_SIG: now also J2.2; no longer LIGHTS.P$1
- net BRAKE_SNS: now also U$3.D17/A3/TOUCH/(SDA0); no longer U$1.1
- net CLK: now also U$3.D14/A0/(SCK0)/PWM; no longer JP2.2
- net CLK_A: now also U$3.D32/A13/SCK1/TX4
- net CLK_B: now also U$3.D13/LED/SCK0
- net GND: now also J8.2; no longer ADD1.S, R17.2, R2.2
- net HAZ_L_SIG: now also J1.2; no longer LIGHTS.P$2
- net HAZ_R_SIG: now also J1.3; no longer LIGHTS.P$3
- net HEADLIGHT_SIG: now also J1.4; no longer LIGHTS.P$4
- net ISOENABLE: now also U$3.D38/A19/SDA1/PWM
- net MISO_A: now also U$3.D1/TOUCH/MISO1/TX1
- net MISO_B: now also U$3.D12/MISO0
- net MOSI_A: now also U$3.D0/TOUCH/MOSI1/RX1
- net MOSI_B: now also U$3.D11/MOSI0
- net PEDAL_SNS: now also U$3.D39/A20
- net REARLIGHT_SIG: now also J1.5; no longer LIGHTS.P$5
- net VDD: no longer ADD1.D, LIGHTS.P$6, LIGHTS.P$7, LIGHTS.P$8
- net µC_GND: no longer R23.2, R24.2, R25.2, U$1.5
Other:
- note removed: "Add. #1"
- note removed: "CLK Jumper"
- note removed: "GPIO BUS"

Commit message: Schematic first version
Parts:
- removed JP1: (no value), jumper:JP1Q
Connections:
- removed net µC_GND: JP1.2
- new net VIPER: J2.3
- net GND: no longer JP1.1
- net HORN: now also J2.4
Changed lines of the file:
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@@
 <part name="TRACO" library="master_library" deviceset="TRACO-TSR-1-2450" device=""/>
 <part name="LM2940" library="master_library" deviceset="LM2940" device="LM" package3d_urn="urn:adsk.eagle:package:8814566/1"/>
-<part name="JP1" library="jumper" library_urn="urn:adsk.eagle:library:252" deviceset="JP1Q" device="" package3d_urn="urn:adsk.eagle:package:15455/1"/>
 <part name="SUPPLY12" library="supply2" library_urn="urn:adsk.eagle:library:372" deviceset="GND" device=""/>
 <part name="SUPPLY13" library="supply2" library_urn="urn:adsk.eagle:library:372" deviceset="GND" device=""/>
@@
 </instance>
 <instance part="LM2940" gate="G$1" x="-85.09" y="108.966" smashed="yes" rot="R90"/>
-<instance part="JP1" gate="A" x="137.16" y="154.94" smashed="yes" rot="R90">
-<attribute name="NAME" x="131.8768" y="157.1752" size="1.778" layer="95" rot="SR0"/>
-<attribute name="VALUE" x="142.24" y="159.385" size="1.778" layer="96" rot="R180"/>
-</instance>
 <instance part="SUPPLY12" gate="GND" x="48.26" y="13.285" smashed="yes"/>
 <instance part="SUPPLY13" gate="GND" x="63.5" y="10.745" smashed="yes"/>
@@
 </segment>
 </net>
-<net name="µC_GND" class="0">
-<segment>
-<pinref part="JP1" gate="A" pin="2"/>
-<wire x1="129.54" y1="154.94" x2="127" y2="154.94" width="0.1524" layer="91"/>
-<label x="114.3" y="154.94" size="1.778" layer="95"/>
-</segment>
-</net>
 <net name="5V_REG" class="0">
 <segment>
@@
 </segment>
 <segment>
-<pinref part="JP1" gate="A" pin="1"/>
-<wire x1="144.78" y1="154.94" x2="147.32" y2="154.94" width="0.1524" layer="91"/>
-<label x="147.32" y="154.94" size="1.778" layer="95"/>
-</segment>
-<segment>
 <pinref part="R5" gate="G$1" pin="2"/>
 <pinref part="SUPPLY18" gate="GND" pin="GND"/>
@@
 <label x="-38.1" y="12.7" size="1.778" layer="95"/>
 </segment>
+<segment>
+<pinref part="J2" gate="G$1" pin="4"/>
+<wire x1="121.92" y1="101.6" x2="127" y2="101.6" width="0.1524" layer="91"/>
+<label x="127" y="101.6" size="1.778" layer="95"/>
+</segment>
 </net>
 <net name="MOSI_SW" class="0">
@@
 </segment>
 </net>
+<net name="VIPER" class="0">
+<segment>
+<pinref part="J2" gate="G$1" pin="3"/>
+<wire x1="101.6" y1="101.6" x2="96.52" y2="101.6" width="0.1524" layer="91"/>
+<label x="91.44" y="101.6" size="1.778" layer="95"/>
+</segment>
+</net>

Commit message: Board layout proposal
Other:
- note added: "Teensy 3.5"
- moved on the sheet: BACK, BRAKE, FRONT, HAZ_L, HAZ_R, HEAD, HORN, J8, LEFT, R18, R19, R20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

Commit message: Board first version
Connections:
- removed net 5V: J7.1
- net 5V_REG: now also J7.1
- net CLK_SW: now also J8.6; no longer J8.4
- net CS: now also J8.4; no longer J8.6
- net MOSI_SW: now also J8.7; no longer J8.3
- net RESET: now also J8.3; no longer J8.7
Changed lines of the file:
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@@
 <label x="187.96" y="116.84" size="1.778" layer="95"/>
+</segment>
+<segment>
+<pinref part="J7" gate="G$1" pin="1"/>
+<wire x1="-25.4" y1="109.22" x2="-33.02" y2="109.22" width="0.1524" layer="91"/>
+<label x="-38.1" y="109.22" size="1.778" layer="95"/>
 </segment>
 </net>
@@
 </segment>
 </net>
-<net name="5V" class="0">
-<segment>
-<pinref part="J7" gate="G$1" pin="1"/>
-<wire x1="-25.4" y1="109.22" x2="-33.02" y2="109.22" width="0.1524" layer="91"/>
-<label x="-38.1" y="109.22" size="1.778" layer="95"/>
-</segment>
-</net>
 <net name="PEDAL_SNS" class="0">
 <segment>
@@
 </net>
 <net name="MOSI_SW" class="0">
+<segment>
+<pinref part="U$3" gate="G$1" pin="D3/SCL2/CAN0TX/PWM"/>
+<wire x1="147.32" y1="38.1" x2="139.7" y2="38.1" width="0.1524" layer="91"/>
+<label x="134.62" y="38.1" size="1.778" layer="95"/>
+</segment>
+<segment>
+<pinref part="J8" gate="G$1" pin="7"/>
+<wire x1="206.502" y1="107.188" x2="200.66" y2="107.188" width="0.1524" layer="91"/>
+<wire x1="200.66" y1="107.188" x2="200.66" y2="109.22" width="0.1524" layer="91"/>
+<label x="187.96" y="109.22" size="1.778" layer="95"/>
+</segment>
+</net>
+<net name="CLK_SW" class="0">
+<segment>
+<pinref part="U$3" gate="G$1" pin="D2/PWM"/>
+<wire x1="147.32" y1="40.64" x2="139.7" y2="40.64" width="0.1524" layer="91"/>
+<label x="134.62" y="40.64" size="1.778" layer="95"/>
+</segment>
+<segment>
+<pinref part="J8" gate="G$1" pin="6"/>
+<wire x1="226.822" y1="109.728" x2="233.68" y2="109.728" width="0.1524" layer="91"/>
+<wire x1="233.68" y1="109.728" x2="233.68" y2="111.76" width="0.1524" layer="91"/>
+<label x="233.68" y="111.76" size="1.778" layer="95"/>
+</segment>
+</net>
+<net name="DC" class="0">
+<segment>
+<pinref part="J8" gate="G$1" pin="5"/>
+<wire x1="206.502" y1="109.728" x2="200.66" y2="109.728" width="0.1524" layer="91"/>
+<wire x1="200.66" y1="109.728" x2="200.66" y2="111.76" width="0.1524" layer="91"/>
+<label x="187.96" y="111.76" size="1.778" layer="95"/>
+</segment>
+<segment>
+<pinref part="U$3" gate="G$1" pin="D5/(MISO)/(TX1)/PWM"/>
+<wire x1="147.32" y1="33.02" x2="139.7" y2="33.02" width="0.1524" layer="91"/>
+<label x="134.62" y="33.02" size="1.778" layer="95"/>
+</segment>
+</net>
+<net name="CS" class="0">
+<segment>
+<pinref part="U$3" gate="G$1" pin="D4/SDA2/CAN0RX/PWM"/>
+<wire x1="147.32" y1="35.56" x2="139.7" y2="35.56" width="0.1524" layer="91"/>
+<label x="134.62" y="35.56" size="1.778" layer="95"/>
+</segment>
+<segment>
+<pinref part="J8" gate="G$1" pin="4"/>
+<wire x1="226.822" y1="112.268" x2="233.68" y2="112.268" width="0.1524" layer="91"/>
+<wire x1="233.68" y1="112.268" x2="233.68" y2="114.3" width="0.1524" layer="91"/>
+<label x="233.68" y="114.3" size="1.778" layer="95"/>
+</segment>
+</net>
+<net name="RESET" class="0">
+<segment>
+<pinref part="U$3" gate="G$1" pin="D6/PWM"/>
+<wire x1="147.32" y1="30.48" x2="139.7" y2="30.48" width="0.1524" layer="91"/>
+<label x="134.62" y="30.48" size="1.778" layer="95"/>
+</segment>
 <segment>
 <pinref part="J8" gate="G$1" pin="3"/>
@@
 <label x="187.96" y="114.3" size="1.778" layer="95"/>
 </segment>
-<segment>
-<pinref part="U$3" gate="G$1" pin="D3/SCL2/CAN0TX/PWM"/>
-<wire x1="147.32" y1="38.1" x2="139.7" y2="38.1" width="0.1524" layer="91"/>
-<label x="134.62" y="38.1" size="1.778" layer="95"/>
-</segment>
-</net>
-<net name="CLK_SW" class="0">
-<segment>
-<pinref part="J8" gate="G$1" pin="4"/>
-<wire x1="226.822" y1="112.268" x2="233.68" y2="112.268" width="0.1524" layer="91"/>
-<wire x1="233.68" y1="112.268" x2="233.68" y2="114.3" width="0.1524" layer="91"/>
-<label x="233.68" y="114.3" size="1.778" layer="95"/>
-</segment>
-<segment>
-<pinref part="U$3" gate="G$1" pin="D2/PWM"/>
-<wire x1="147.32" y1="40.64" x2="139.7" y2="40.64" width="0.1524" layer="91"/>
-<label x="134.62" y="40.64" size="1.778" layer="95"/>
-</segment>
-</net>
-<net name="DC" class="0">
-<segment>
-<pinref part="J8" gate="G$1" pin="5"/>
-<wire x1="206.502" y1="109.728" x2="200.66" y2="109.728" width="0.1524" layer="91"/>
-<wire x1="200.66" y1="109.728" x2="200.66" y2="111.76" width="0.1524" layer="91"/>
-<label x="187.96" y="111.76" size="1.778" layer="95"/>
-</segment>
-<segment>
-<pinref part="U$3" gate="G$1" pin="D5/(MISO)/(TX1)/PWM"/>
-<wire x1="147.32" y1="33.02" x2="139.7" y2="33.02" width="0.1524" layer="91"/>
-<label x="134.62" y="33.02" size="1.778" layer="95"/>
-</segment>
-</net>
-<net name="CS" class="0">
-<segment>
-<pinref part="J8" gate="G$1" pin="6"/>
-<wire x1="226.822" y1="109.728" x2="233.68" y2="109.728" width="0.1524" layer="91"/>
-<wire x1="233.68" y1="109.728" x2="233.68" y2="111.76" width="0.1524" layer="91"/>
-<label x="233.68" y="111.76" size="1.778" layer="95"/>
-</segment>
-<segment>
-<pinref part="U$3" gate="G$1" pin="D4/SDA2/CAN0RX/PWM"/>
-<wire x1="147.32" y1="35.56" x2="139.7" y2="35.56" width="0.1524" layer="91"/>
-<label x="134.62" y="35.56" size="1.778" layer="95"/>
-</segment>
-</net>
-<net name="RESET" class="0">
-<segment>
-<pinref part="J8" gate="G$1" pin="7"/>
-<wire x1="206.502" y1="107.188" x2="200.66" y2="107.188" width="0.1524" layer="91"/>
-<wire x1="200.66" y1="107.188" x2="200.66" y2="109.22" width="0.1524" layer="91"/>
-<label x="187.96" y="109.22" size="1.778" layer="95"/>
-</segment>
-<segment>
-<pinref part="U$3" gate="G$1" pin="D6/PWM"/>
-<wire x1="147.32" y1="30.48" x2="139.7" y2="30.48" width="0.1524" layer="91"/>
-<label x="134.62" y="30.48" size="1.778" layer="95"/>
-</segment>
-</net>
+</net>

Commit message: VIPER misspelling corrected
Connections:
- removed net VIPER: J2.3
- net WIPER: now also J2.3
Changed lines of the file:
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@@
 <label x="43.18" y="91.44" size="1.778" layer="95"/>
+</segment>
+<segment>
+<pinref part="J2" gate="G$1" pin="3"/>
+<wire x1="101.6" y1="101.6" x2="96.52" y2="101.6" width="0.1524" layer="91"/>
+<label x="91.44" y="101.6" size="1.778" layer="95"/>
 </segment>
 </net>
@@
 </segment>
 </net>
-<net name="VIPER" class="0">
-<segment>
-<pinref part="J2" gate="G$1" pin="3"/>
-<wire x1="101.6" y1="101.6" x2="96.52" y2="101.6" width="0.1524" layer="91"/>
-<label x="91.44" y="101.6" size="1.778" layer="95"/>
-</segment>
-</net>

Commit message: Widen the traces of independent 12V and indipendent ground
Changed lines of the file:
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@@
 <segment>
 <pinref part="R8" gate="G$1" pin="1"/>
-<label x="-55.525228125" y="27.963965625" size="1.778" layer="95"/>
+<label x="-58.065228125" y="27.963965625" size="1.778" layer="95"/>
 <wire x1="-55.88" y1="28.0358625" x2="-54.85544375" y2="27.963965625" width="0.1524" layer="91"/>
 </segment>

Commit message: Added voltage divider so that Teensy 3.5 sees Wiper and Horn are turned on
Parts:
- added R10, R2: 3K, master_library:R-US_R0805
- added R11, R3: 5K, master_library:R-US_R0805
Connections:
- new net HORN_IN: R10.1, R11.2, U$3.D22/A8/TOUCH/PWM
- new net WIPER_IN: R2.1, R3.2, U$3.D23/A9/TOUCH/PWM
- net GND: now also R11.1, R3.1
- net H4: now also R2.2
- net H9: now also R10.2
Other:
- moved on the sheet: J7
Changed lines of the file:
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@@
 <part name="U$6" library="AUX Lib" deviceset="TE_CON_OJE-SH-112DM,095\" device=""/>
 <part name="J8" library="AUX Lib" deviceset="SS-6488-NF-A431" device=""/>
+<part name="R2" library="master_library" deviceset="R-US_" device="R0805" package3d_urn="urn:adsk.eagle:package:2274104/1" value="3K"/>
+<part name="R3" library="master_library" deviceset="R-US_" device="R0805" package3d_urn="urn:adsk.eagle:package:2274104/1" value="5K"/>
+<part name="R10" library="master_library" deviceset="R-US_" device="R0805" package3d_urn="urn:adsk.eagle:package:2274104/1" value="3K"/>
+<part name="R11" library="master_library" deviceset="R-US_" device="R0805" package3d_urn="urn:adsk.eagle:package:2274104/1" value="5K"/>
 </parts>
 <sheets>
@@
 <attribute name="VALUE" x="21.59" y="177.8" size="1.778" layer="96" align="center-left"/>
 </instance>
-<instance part="J7" gate="G$1" x="-25.4" y="109.22" smashed="yes">
-<attribute name="NAME" x="-8.89" y="116.84" size="1.778" layer="95" align="center-left"/>
-<attribute name="VALUE" x="-8.89" y="114.3" size="1.778" layer="96" align="center-left"/>
+<instance part="J7" gate="G$1" x="-25.4" y="129.54" smashed="yes">
+<attribute name="NAME" x="-8.89" y="137.16" size="1.778" layer="95" align="center-left"/>
+<attribute name="VALUE" x="-8.89" y="134.62" size="1.778" layer="96" align="center-left"/>
 </instance>
 <instance part="U$5" gate="G$1" x="71.12" y="106.68" smashed="yes">
@@
 <attribute name="NAME" x="223.012" y="122.428" size="1.778" layer="95" align="center-left"/>
 <attribute name="VALUE" x="223.012" y="119.888" size="1.778" layer="96" align="center-left"/>
+</instance>
+<instance part="R2" gate="G$1" x="-2.54" y="109.22" smashed="yes">
+<attribute name="NAME" x="-6.35" y="110.7186" size="1.778" layer="95"/>
+<attribute name="VALUE" x="-6.35" y="105.918" size="1.778" layer="96"/>
+</instance>
+<instance part="R3" gate="G$1" x="-27.94" y="109.22" smashed="yes">
+<attribute name="NAME" x="-31.75" y="110.7186" size="1.778" layer="95"/>
+<attribute name="VALUE" x="-31.75" y="105.918" size="1.778" layer="96"/>
+</instance>
+<instance part="R10" gate="G$1" x="-2.54" y="96.52" smashed="yes">
+<attribute name="NAME" x="-6.35" y="98.0186" size="1.778" layer="95"/>
+<attribute name="VALUE" x="-6.35" y="93.218" size="1.778" layer="96"/>
+</instance>
+<instance part="R11" gate="G$1" x="-27.94" y="96.52" smashed="yes">
+<attribute name="NAME" x="-31.75" y="98.0186" size="1.778" layer="95"/>
+<attribute name="VALUE" x="-31.75" y="93.218" size="1.778" layer="96"/>
 </instance>
 </instances>
@@
 <wire x1="35.56" y1="114.3" x2="35.56" y2="119.38" width="0.1524" layer="91"/>
 <label x="33.02" y="119.38" size="1.778" layer="95"/>
+</segment>
+<segment>
+<pinref part="R2" gate="G$1" pin="2"/>
+<wire x1="2.54" y1="109.22" x2="7.62" y2="109.22" width="0.1524" layer="91"/>
+<label x="7.62" y="109.22" size="1.778" layer="95"/>
 </segment>
 </net>
@@
 <segment>
 <pinref part="J7" gate="G$1" pin="1"/>
-<wire x1="-25.4" y1="109.22" x2="-33.02" y2="109.22" width="0.1524" layer="91"/>
-<label x="-38.1" y="109.22" size="1.778" layer="95"/>
+<wire x1="-25.4" y1="129.54" x2="-33.02" y2="129.54" width="0.1524" layer="91"/>
+<label x="-38.1" y="129.54" size="1.778" layer="95"/>
 </segment>
 </net>
@@
 <segment>
 <pinref part="J7" gate="G$1" pin="3"/>
-<wire x1="-25.4" y1="106.68" x2="-33.02" y2="106.68" width="0.1524" layer="91"/>
-<label x="-38.1" y="106.68" size="1.778" layer="95"/>
+<wire x1="-25.4" y1="127" x2="-33.02" y2="127" width="0.1524" layer="91"/>
+<label x="-38.1" y="127" size="1.778" layer="95"/>
 </segment>
 <segment>
@@
 <label x="233.68" y="116.84" size="1.778" layer="95"/>
 </segment>
+<segment>
+<pinref part="R3" gate="G$1" pin="1"/>
+<wire x1="-33.02" y1="109.22" x2="-38.1" y2="109.22" width="0.1524" layer="91"/>
+<label x="-38.1" y="109.22" size="1.778" layer="95"/>
+</segment>
+<segment>
+<pinref part="R11" gate="G$1" pin="1"/>
+<wire x1="-33.02" y1="96.52" x2="-38.1" y2="96.52" width="0.1524" layer="91"/>
+<label x="-38.1" y="96.52" size="1.778" layer="95"/>
+</segment>
 </net>
 <net name="N$8" class="0">
@@
 <segment>
 <pinref part="J7" gate="G$1" pin="2"/>
-<wire x1="-5.08" y1="109.22" x2="5.08" y2="109.22" width="0.1524" layer="91"/>
-<label x="-2.54" y="106.68" size="1.778" layer="95"/>
+<wire x1="-5.08" y1="129.54" x2="5.08" y2="129.54" width="0.1524" layer="91"/>
+<label x="-2.54" y="127" size="1.778" layer="95"/>
 </segment>
 <segment>
@@
 <wire x1="66.04" y1="114.3" x2="66.04" y2="119.38" width="0.1524" layer="91"/>
 <label x="63.5" y="119.38" size="1.778" layer="95"/>
+</segment>
+<segment>
+<pinref part="R10" gate="G$1" pin="2"/>
+<wire x1="2.54" y1="96.52" x2="7.62" y2="96.52" width="0.1524" layer="91"/>
+<label x="7.62" y="96.52" size="1.778" layer="95"/>
 </segment>
 </net>
@@
 </segment>
 </net>
+<net name="WIPER_IN" class="0">
+<segment>
+<pinref part="U$3" gate="G$1" pin="D23/A9/TOUCH/PWM"/>
+<wire x1="218.44" y1="40.64" x2="226.06" y2="40.64" width="0.1524" layer="91"/>
+<label x="226.06" y="40.64" size="1.778" layer="95"/>
+</segment>
+<segment>
+<pinref part="R2" gate="G$1" pin="1"/>
+<pinref part="R3" gate="G$1" pin="2"/>
+<wire x1="-7.62" y1="109.22" x2="-15.24" y2="109.22" width="0.1524" layer="91"/>
+<wire x1="-15.24" y1="109.22" x2="-22.86" y2="109.22" width="0.1524" layer="91"/>
+<wire x1="-15.24" y1="109.22" x2="-15.24" y2="101.6" width="0.1524" layer="91"/>
+<junction x="-15.24" y="109.22"/>
+<label x="-15.24" y="101.6" size="1.778" layer="95"/>
+</segment>
+</net>
+<net name="HORN_IN" class="0">
+<segment>
+<pinref part="U$3" gate="G$1" pin="D22/A8/TOUCH/PWM"/>
+<wire x1="218.44" y1="38.1" x2="226.06" y2="38.1" width="0.1524" layer="91"/>
+<label x="226.06" y="38.1" size="1.778" layer="95"/>
+</segment>
+<segment>
+<pinref part="R10" gate="G$1" pin="1"/>
+<pinref part="R11" gate="G$1" pin="2"/>
+<wire x1="-7.62" y1="96.52" x2="-15.24" y2="96.52" width="0.1524" layer="91"/>
+<wire x1="-15.24" y1="96.52" x2="-22.86" y2="96.52" width="0.1524" layer="91"/>
+<wire x1="-15.24" y1="96.52" x2="-15.24" y2="88.9" width="0.1524" layer="91"/>
+<junction x="-15.24" y="96.52"/>
+<label x="-15.24" y="88.9" size="1.778" layer="95"/>
+</segment>
+</net>
